Commit message: Merge branch 'calibrated_camera_setup'

File: src/viola_moveit_config/config/camera_with_stand.xacro (robot description, xacro)
@@ -1,31 +1,21 @@
 <?xml version="1.0"?>
 <robot xmlns:xacro="http://ros.org/wiki/xacro" >
+    <!-- Variables -->
+    <xacro:property name="pi_val" value="3.1415926535"/>
+    <!-- Materials -->
+    <material name="gray">
+        <color rgba="0.5 0.5 0.5 1" />
+    </material>
     <xacro:macro name="camera_with_stand" params="camera_pos_z
-                                                  camera_roll:=0.0 camera_pitch:=0.0 camera_yaw:=0.0
-                                                  camera_type:=realsense">
-        <!-- Variables -->
-        <xacro:property name="pi_val" value="3.1415926535"/>
-        <!-- Materials -->
-        <material name="gray">
-            <color rgba="0.5 0.5 0.5 1" />
-        </material>
+                                                  camera_roll:=0.0
+                                                  camera_pitch:=0.0
+                                                  camera_yaw:=0.0
+                                                  camera_name:=camera">
         <!-- Include realsense urdf macro -->
-        <xacro:if value="${camera_type == 'realsense'}">
-            <xacro:include filename="$(find realsense2_description)/urdf/_d435i.urdf.xacro"/>
-        </xacro:if>
+        <xacro:include filename="$(find realsense2_description)/urdf/_d435i.urdf.xacro"/>
         <!-- Links -->
+        <link name="camera_connection_link"/>
+        <link name="camera_base_link"/>
         <link name="camera_mount_link"/>
-        <link name="camera_base_link"/>
-        <xacro:if value="${camera_type != 'realsense'}">
-            <link name="camera_link">
-                <visual>
-                    <origin xyz="0 0 -0.015" rpy="0 0 0"/>
-                    <geometry>
-                        <cylinder radius="0.03" length="0.03"/>
-                    </geometry>
-                    <material name="gray"/>
-                </visual>
-            </link>
-        </xacro:if>
         <link name="camera_holder_upper_arm_link">
             <visual>
@@ -68,22 +58,18 @@
         </link>
         <!-- Joints -->
-        <joint name="camera_mount_camera_base_joint" type="fixed">
-            <parent link="camera_mount_link"/>
+        <xacro:sensor_d435i parent="camera_connection_link" name="${camera_name}" use_nominal_extrinsics="true" >
+            <origin xyz="0 0 0" rpy="${camera_roll} ${camera_pitch} ${camera_yaw}"/>
+        </xacro:sensor_d435i>
+        <joint name="camera_connection_to_camera_base_joint" type="fixed">
+            <parent link="camera_connection_link"/>
             <child link="camera_base_link"/>
-            <origin xyz="0 0 0" rpy="${camera_roll} ${camera_pitch} ${camera_yaw}"/>
+            <origin xyz="-0.0095 0 0.0125" rpy="0 0 0"/>
         </joint>
-        <xacro:if value="${camera_type == 'realsense'}">
-            <xacro:sensor_d435i parent="camera_base_link" use_nominal_extrinsics="true" >
-                <origin xyz="0.0095 0 -0.0125" rpy="0 0 0"/>
-            </xacro:sensor_d435i>
-        </xacro:if>
-        <xacro:if value="${camera_type != 'realsense'}">
-            <joint name="camera_base_to_camera_joint" type="fixed">
-                <parent link="camera_base_link"/>
-                <child link="camera_link"/>
-                <origin xyz="0 0 0" rpy="0 ${pi_val/2} 0"/>
-            </joint>
-        </xacro:if>
-        <joint name="camera_base_to_upper_arm_joint" type="fixed">
+        <joint name="camera_base_to_camera_mount_joint" type="fixed">
+            <parent link="camera_base_link"/>
+            <child link="camera_mount_link"/>
+            <origin xyz="0 0 0" rpy="0 0 0"/>
+        </joint>
+        <joint name="camera_mount_to_upper_arm_joint" type="fixed">
             <parent link="camera_mount_link"/>
             <child link="camera_holder_upper_arm_link"/>

File: src/viola_moveit_config/config/viola_description.urdf.xacro (robot description, xacro)
@@ -3,7 +3,8 @@
     <!-- Arguments -->
     <xacro:arg name="initial_positions_file" default="initial_positions.yaml" />
-    <xacro:arg name="launch_calibration" default="true" />
+    <xacro:arg name="launch_calibration" default="false" />
+    <xacro:arg name="use_camera_calibration" default="false" />
     <xacro:arg name="launch_camera" default="false" />
-    <xacro:arg name="camera_type" default="realsense" />
+    <xacro:arg name="camera_name" default="camera" />
     <xacro:arg name="camera_pos_x" default="0.4" />
     <xacro:arg name="camera_pos_y" default="0.0" />
@@ -17,14 +18,16 @@
     <xacro:include filename="viola_description.ros2_control.xacro" />
     <xacro:viola_description_ros2_control name="FakeSystem" initial_positions_file="$(arg initial_positions_file)"/>
-    <!-- Conditionally include camera-->
-    <xacro:if value="$(eval launch_camera)">
+    <!-- Conditionally include measured camera pose-->
+    <xacro:if value="$(eval launch_camera and not use_camera_calibration)">
         <xacro:include filename="$(find viola_moveit_config)/config/camera_with_stand.xacro"/>
         <xacro:camera_with_stand camera_pos_z="$(arg camera_pos_z)"
-                                 camera_roll="$(arg camera_pos_roll)" camera_pitch="$(arg camera_pos_pitch)" camera_yaw="$(arg camera_pos_yaw)"
-                                 camera_type="$(arg camera_type)" />
+                                 camera_roll="$(arg camera_pos_roll)"
+                                 camera_pitch="$(arg camera_pos_pitch)"
+                                 camera_yaw="$(arg camera_pos_yaw)"
+                                 camera_name="$(arg camera_name)" />
         <!-- Connect camera to robot base -->
-        <joint name="base_link_camera_mount_joint" type="fixed">
+        <joint name="base_link_to_camera_connection_joint" type="fixed">
             <parent link="base_link"/>
-            <child link="camera_mount_link"/>
+            <child link="camera_connection_link"/>
             <origin xyz="$(arg camera_pos_x) $(arg camera_pos_y) $(arg camera_pos_z)"
                     rpy="0 0 0"/>
